Commit message: adapt system for joint limits

File: src/arctos_description/urdf/arctos_urdf.xacro (robot description, xacro)
@@ -2,6 +2,9 @@
 <robot name="arctos" xmlns:xacro="http://www.ros.org/wiki/xacro">
 <xacro:include filename="$(find arctos_description)/urdf/materials.xacro" />
-<xacro:include filename="$(find arctos_description)/urdf/arctos_urdf.trans" />
-<xacro:include filename="$(find arctos_description)/urdf/arctos_urdf.gazebo" />
+<xacro:arg name="legacy_control" default="true"/>
+<xacro:if value="$(arg legacy_control)">
+  <xacro:include filename="$(find arctos_description)/urdf/arctos_urdf.trans" />
+  <xacro:include filename="$(find arctos_description)/urdf/arctos_urdf.gazebo" />
+</xacro:if>
 <link name="world"/>
 <joint name="base_joint" type="fixed">
@@ -266,5 +269,7 @@
   <limit upper="0.015" lower="0.0" effort="100" velocity="100"/>
 </joint>
-<xacro:include filename="$(find arctos_hardware_interface)/ros2_control/arctos.ros2_control.xacro" />
-<xacro:arctos_ros2_control name="arctos"/>
+<xacro:if value="$(arg legacy_control)">
+  <xacro:include filename="$(find arctos_hardware_interface)/ros2_control/arctos.ros2_control.xacro" />
+  <xacro:arctos_ros2_control name="arctos"/>
+</xacro:if>
 </robot>

File: src/arctos_moveit_config/config/arctos_urdf.ros2_control.xacro (robot description, xacro)
@@ -1,65 +1,29 @@
 <?xml version="1.0"?>
 <robot xmlns:xacro="http://www.ros.org/wiki/xacro">
-    <xacro:macro name="arctos_urdf_ros2_control" params="name initial_positions_file">
-        <xacro:property name="initial_positions" value="${load_yaml(initial_positions_file)['initial_positions']}"/>
-        <ros2_control type="system">
-	    <hardware>
-	      <plugin>arctos_interface/ArctosInterface</plugin>
-	    </hardware>
-	    <joint name="joint1">
-	      <command_interface name="position"/>
-	      <state_interface name="position">
-		<param name="initial_value">0.0</param>
-	      </state_interface>
-	      <state_interface name="velocity">
-		<param name="initial_value">0.0</param>
-	      </state_interface>
-	    </joint>
-	    <joint name="joint2">
-	      <command_interface name="position"/>
-	      <state_interface name="position">
-		<param name="initial_value">0.0</param>
-	      </state_interface>
-	      <state_interface name="velocity">
-		<param name="initial_value">0.0</param>
-	      </state_interface>
-	    </joint>
-	    <joint name="joint3">
-	      <command_interface name="position"/>
-	      <state_interface name="position">
-		<param name="initial_value">0.0</param>
-	      </state_interface>
-	      <state_interface name="velocity">
-		<param name="initial_value">0.0</param>
-	      </state_interface>
-	    </joint>
-	    <joint name="joint4">
-	      <command_interface name="position"/>
-	      <state_interface name="position">
-		<param name="initial_value">0.0</param>
-	      </state_interface>
-	      <state_interface name="velocity">
-		<param name="initial_value">0.0</param>
-	      </state_interface>
-	    </joint>
-	    <joint name="joint5">
-	      <command_interface name="position"/>
-	      <state_interface name="position">
-		<param name="initial_value">0.0</param>
-	      </state_interface>
-	      <state_interface name="velocity">
-		<param name="initial_value">0.0</param>
-	      </state_interface>
-	    </joint>
-	    <joint name="joint6">
-	      <command_interface name="position"/>
-	      <state_interface name="position">
-		<param name="initial_value">0.0</param>
-	      </state_interface>
-	      <state_interface name="velocity">
-		<param name="initial_value">0.0</param>
-	      </state_interface>
-	    </joint>
-	</ros2_control>
+  <!-- Kinematic simulation only: no motor transport or physical dynamics. -->
+  <xacro:macro name="arctos_urdf_ros2_control" params="name initial_positions_file">
+    <xacro:property name="initial_positions" value="${xacro.load_yaml(initial_positions_file)['initial_positions']}"/>
+    <xacro:macro name="mock_joint" params="joint_name">
+      <joint name="${joint_name}">
+        <command_interface name="position"/>
+        <state_interface name="position">
+          <param name="initial_value">${initial_positions[joint_name]}</param>
+        </state_interface>
+        <state_interface name="velocity"/>
+      </joint>
     </xacro:macro>
+    <ros2_control name="${name}" type="system">
+      <hardware>
+        <plugin>mock_components/GenericSystem</plugin>
+      </hardware>
+      <xacro:mock_joint joint_name="joint_1"/>
+      <xacro:mock_joint joint_name="joint_2"/>
+      <xacro:mock_joint joint_name="joint_3"/>
+      <xacro:mock_joint joint_name="joint_4"/>
+      <xacro:mock_joint joint_name="joint_5"/>
+      <xacro:mock_joint joint_name="joint_6"/>
+      <xacro:mock_joint joint_name="jaw1"/>
+      <xacro:mock_joint joint_name="jaw2"/>
+    </ros2_control>
+  </xacro:macro>
 </robot>

File: src/arctos_moveit_config/config/arctos_urdf.urdf.xacro (robot description, xacro)
@@ -3,5 +3,6 @@
     <xacro:arg name="initial_positions_file" default="initial_positions.yaml" />
     <!-- Import arctos_urdf urdf file -->
-    <xacro:include filename="$(find arctos_description)/urdf/arctos.urdf" />
+    <xacro:arg name="legacy_control" default="false"/>
+    <xacro:include filename="$(find arctos_description)/urdf/arctos_urdf.xacro" />
     <!-- Import control_xacro -->
     <xacro:include filename="arctos_urdf.ros2_control.xacro" />
